File: pico1mhz.kicad_pcb (KiCad board)
At the start: 2 copper layers, 116 x 77.4 mm, 18 parts, among them J1 Conn_02x17_Odd_Even, J2 Conn_02x17_Odd_Even, Q1 BSS138, Q2 BSS138, Q3 BSS138, Q4 BSS138, Q5 BSS138, Q6 BSS138, Q7 BSS138, U1 Pico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

Commit message: Smaller, less than 100mm
Parts:
- moved RN1 41.3 mm to (135.4, 119.7)
- moved H4 10.8 mm to (185.2, 139.8)
- moved H2 10.4 mm to (185.6, 71.4)
- moved J2 8.75 mm to (184.7, 118.0)
- moved H1 5.10 mm to (94.6, 72.0)
- moved H3 3.64 mm to (93.0, 139.0)
Routing:
- net +3.3V: track 144.5 -> 130.5 mm
- net /R/~{W}_L: track 127.2 -> 116.2 mm
- net /A4: track 44.3 -> 33.7 mm
- net /A6: track 44.2 -> 33.8 mm
- net /A2: track 44.2 -> 33.8 mm
- net /A0: track 44.2 -> 33.8 mm
- net /D3: track 46.4 -> 36.0 mm
- net /D7: track 46.4 -> 36.0 mm
- net /D5: track 46.4 -> 37.6 mm
- net /D1: track 46.4 -> 37.6 mm
- net /~{NMI}: track 52.1 -> 43.4 mm
- net /A1: track 41.2 -> 32.5 mm
- net /R/~{W}: track 54.1 -> 45.3 mm
- net /FRED: track 51.2 -> 42.5 mm
- net /A7: track 41.2 -> 32.5 mm
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Other:
- board size 116 x 77.4 mm -> 99 x 76.8 mm
- board text removed: "V"

Commit message: fixup after size change
Routing:
- net +3.3V: track 130.5 -> 138.9 mm
- net /A4: track 33.7 -> 35.6 mm
- net /D7: track 36.0 -> 37.6 mm
- net /A0: track 33.8 -> 35.5 mm
- net /D3: track 36.0 -> 37.6 mm
- net /A6: track 33.8 -> 35.5 mm
- net /A2: track 33.8 -> 35.5 mm
Changed lines of the file:
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@@
+	)
+	(segment
+		(start 151.6 81.45)
+		(end 166.534554 81.45)
+		(width 0.2)
+		(layer "B.Cu")
+		(net 8)
+	)
+	(segment
+		(start 170.541314 83.5898)
+		(end 171.691114 82.44)
+		(width 0.2)
+		(layer "B.Cu")
+		(net 8)
+	)
+	(segment
+		(start 168.674354 83.5898)
+		(end 170.541314 83.5898)
+		(width 0.2)
+		(layer "B.Cu")
+		(net 8)
 	)
 	(segment
@@
 	)
 	(segment
-		(start 168.674354 83.5898)
-		(end 170.540114 83.5898)
-		(width 0.2)
-		(layer "B.Cu")
-		(net 8)
-	)
-	(segment
-		(start 151.6 81.45)
-		(end 166.534554 81.45)
-		(width 0.2)
-		(layer "B.Cu")
-		(net 8)
-	)
-	(segment
 		(start 169.151114 100.22)
 		(end 170.302114 99.069)
@@
 	)
 	(segment
+		(start 170.541314 78.5098)
+		(end 171.691114 77.36)
+		(width 0.2)
+		(layer "B.Cu")
+		(net 14)
+	)
+	(segment
+		(start 166.534554 76.37)
+		(end 168.674354 78.5098)
+		(width 0.2)
+		(layer "B.Cu")
+		(net 14)
+	)
+	(segment
 		(start 151.6 76.37)
 		(end 166.534554 76.37)
@@
 	(segment
 		(start 168.674354 78.5098)
-		(end 170.540114 78.5098)
-		(width 0.2)
-		(layer "B.Cu")
-		(net 14)
-	)
-	(segment
-		(start 166.534554 76.37)
-		(end 168.674354 78.5098)
+		(end 170.541314 78.5098)
 		(width 0.2)
 		(layer "B.Cu")
@@
 	)
 	(segment
+		(start 170.391114 81.2)
+		(end 171.691114 79.9)
+		(width 0.2)
+		(layer "B.Cu")
+		(net 16)
+	)
+	(segment
+		(start 166.188 78.91)
+		(end 168.478 81.2)
+		(width 0.2)
+		(layer "B.Cu")
+		(net 16)
+	)
+	(segment
+		(start 168.478 81.2)
+		(end 170.391114 81.2)
+		(width 0.2)
+		(layer "B.Cu")
+		(net 16)
+	)
+	(segment
 		(start 151.6 78.91)
 		(end 166.188 78.91)
@@
 	)
 	(segment
-		(start 168.478 81.2)
-		(end 170.389914 81.2)
-		(width 0.2)
-		(layer "B.Cu")
-		(net 16)
-	)
-	(segment
-		(start 166.188 78.91)
-		(end 168.478 81.2)
-		(width 0.2)
-		(layer "B.Cu")
-		(net 16)
-	)
-	(segment
 		(start 169.151114 105.3)
 		(end 170.302114 104.149)
@@
 	)
 	(segment
+		(start 151.6 83.99)
+		(end 166.534554 83.99)
+		(width 0.2)
+		(layer "B.Cu")
+		(net 19)
+	)
+	(segment
 		(start 168.674354 86.1298)
-		(end 170.540114 86.1298)
+		(end 170.541314 86.1298)
+		(width 0.2)
+		(layer "B.Cu")
+		(net 19)
+	)
+	(segment
+		(start 170.541314 86.1298)
+		(end 171.691114 84.98)
 		(width 0.2)
 		(layer "B.Cu")
@@
 	)
 	(segment
-		(start 151.6 83.99)
-		(end 166.534554 83.99)
-		(width 0.2)
-		(layer "B.Cu")
-		(net 19)
-	)
-	(segment
 		(start 171.691114 92.6)
 		(end 172.842114 93.751)
@@
 	(segment
 		(start 161.112154 101.55)
+		(end 151.8 101.55)
+		(width 0.2)
+		(layer "B.Cu")
+		(net 20)
+	)
+	(segment
+		(start 171.691114 92.6)
+		(end 170.541314 93.7498)
+		(width 0.2)
+		(layer "B.Cu")
+		(net 20)
+	)
+	(segment
+		(start 168.912354 93.7498)
+		(end 161.112154 101.55)
+		(width 0.2)
+		(layer "B.Cu")
+		(net 20)
+	)
+	(segment
+		(start 170.541314 93.7498)
 		(end 168.912354 93.7498)
-		(width 0.2)
-		(layer "B.Cu")
-		(net 20)
-	)
-	(segment
-		(start 151.8 101.55)
-		(end 161.112154 101.55)
-		(width 0.2)
-		(layer "B.Cu")
-		(net 20)
-	)
-	(segment
-		(start 168.912354 93.7498)
-		(end 170.540114 93.7498)
 		(width 0.2)
 		(layer "B.Cu")
@@
 	)
 	(segment
+		(start 170.541314 88.6698)
+		(end 171.691114 87.52)
+		(width 0.2)
+		(layer "B.Cu")
+		(net 22)
+	)
+	(segment
 		(start 168.912354 88.6698)
-		(end 170.540114 88.6698)
+		(end 170.541314 88.6698)
 		(width 0.2)
 		(layer "B.Cu")
@@
 	)
 	(segment
+		(start 135.4 119.72)
+		(end 135.4 115.6)
+		(width 0.5)
+		(layer "F.Cu")
+		(net 52)
+	)
+	(segment
 		(start 144.2 140.8)
 		(end 144.2 137.90674)
@@
 		(width 0.5)
 		(layer "F.Cu")
+		(net 52)
+	)
+	(segment
+		(start 135.4 115.6)
+		(end 138.4 112.6)
+		(width 0.5)
+		(layer "F.Cu")
